File: HW2_HW3/Circuit/ME433_sunyue.brd (EAGLE design)
At the start: 50 x 50 mm, 26 parts

Commit message: HW2_HW3
Routing:
- net B15: track 31.8 -> 30.7 mm
- net 5V: track 84.2 -> 83.2 mm
- net MCLR: track 95.6 -> 94.8 mm
Other:
- board text added: "Sun"
- board text added: "Yue"
- board text removed: "NU Yue Sun"
Changed lines of the file:
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@@
 <setting verticaltext="up"/>
 </settings>
-<grid distance="0.025" unitdist="inch" unit="inch" style="lines" multiple="1" display="no" altdistance="0.00625" altunitdist="inch" altunit="inch"/>
+<grid distance="0.025" unitdist="inch" unit="mm" style="lines" multiple="1" display="no" altdistance="0.00625" altunitdist="inch" altunit="mm"/>
 <layers>
 <layer number="1" name="Top" color="4" fill="1" visible="yes" active="yes"/>
@@
 <text x="33.02" y="44.45" size="0.8128" layer="27">RESET</text>
 <text x="14.9225" y="13.6525" size="0.8128" layer="27" rot="R90">8MHz</text>
-<text x="10.795" y="12.065" size="1.778" layer="27" rot="R90">PIC32MX250F128B</text>
-<text x="13.97" y="19.05" size="1.778" layer="27" rot="R90">NU   Yue Sun</text>
+<text x="10.795" y="15.24" size="1.4224" layer="27" rot="R90">PIC32MX250F128B</text>
+<text x="12.065" y="27.94" size="1.4224" layer="27" rot="R270">Yue</text>
+<text x="13.335" y="29.21" size="1.4224" layer="27" rot="R90">Sun</text>
 </plain>
 <attributes>
@@
 </class>
 </classes>
-<designrules name="default">
+<designrules name="SeeedStudio_2layer_DRU_no_angle_20140221">
 <description language="de">&lt;b&gt;EAGLE Design Rules&lt;/b&gt;
 &lt;p&gt;
@@
 necessary adjustments and save your customized
 design rules under a new name.</description>
+<description language="zh">&lt;b&gt;Seeed Studio EAGLE Design Rules&lt;/b&gt;
+</description>
 <param name="layerSetup" value="(1*16)"/>
-<param name="mtCopper" value="0.035mm 0.035mm 0.035mm 0.035mm 0.035mm 0.035mm 0.035mm 0.035mm 0.035mm 0.035mm 0.035mm 0.035mm 0.035mm 0.035mm 0.035mm 0.035mm"/>
-<param name="mtIsolate" value="1.5mm 0.15mm 0.2mm 0.15mm 0.2mm 0.15mm 0.2mm 0.15mm 0.2mm 0.15mm 0.2mm 0.15mm 0.2mm 0.15mm 0.2mm"/>
-<param name="mdWireWire" value="8mil"/>
-<param name="mdWirePad" value="8mil"/>
-<param name="mdWireVia" value="8mil"/>
-<param name="mdPadPad" value="8mil"/>
-<param name="mdPadVia" value="8mil"/>
-<param name="mdViaVia" value="8mil"/>
-<param name="mdSmdPad" value="8mil"/>
-<param name="mdSmdVia" value="8mil"/>
-<param name="mdSmdSmd" value="8mil"/>
+<param name="mtCopper" value="0.035mm 0.0175mm 0.035mm 0.035mm 0.035mm 0.035mm 0.035mm 0.035mm 0.035mm 0.035mm 0.035mm 0.035mm 0.035mm 0.035mm 0.0175mm 0.035mm"/>
+<param name="mtIsolate" value="1.5mm 1.1mm 0.2mm 0.15mm 0.2mm 0.15mm 0.2mm 0.15mm 0.2mm 0.15mm 0.2mm 0.15mm 0.2mm 0.15mm 0.2mm"/>
+<param name="mdWireWire" value="6mil"/>
+<param name="mdWirePad" value="6mil"/>
+<param name="mdWireVia" value="6mil"/>
+<param name="mdPadPad" value="6mil"/>
+<param name="mdPadVia" value="6mil"/>
+<param name="mdViaVia" value="6mil"/>
+<param name="mdSmdPad" value="0mil"/>
+<param name="mdSmdVia" value="0mil"/>
+<param name="mdSmdSmd" value="0mil"/>
 <param name="mdViaViaSameLayer" value="8mil"/>
 <param name="mnLayersViaInSmd" value="2"/>
-<param name="mdCopperDimension" value="40mil"/>
-<param name="mdDrill" value="8mil"/>
+<param name="mdCopperDimension" value="10mil"/>
+<param name="mdDrill" value="10mil"/>
 <param name="mdSmdStop" value="0mil"/>
-<param name="msWidth" value="10mil"/>
-<param name="msDrill" value="24mil"/>
-<param name="msMicroVia" value="9.99mm"/>
+<param name="msWidth" value="6mil"/>
+<param name="msDrill" value="12mil"/>
+<param name="msMicroVia" value="12mil"/>
 <param name="msBlindViaRatio" value="0.5"/>
 <param name="rvPadTop" value="0.25"/>
@@
 <param name="rlMinPadBottom" value="10mil"/>
 <param name="rlMaxPadBottom" value="20mil"/>
-<param name="rlMinViaOuter" value="8mil"/>
+<param name="rlMinViaOuter" value="6mil"/>
 <param name="rlMaxViaOuter" value="20mil"/>
-<param name="rlMinViaInner" value="8mil"/>
+<param name="rlMinViaInner" value="6mil"/>
 <param name="rlMaxViaInner" value="20mil"/>
 <param name="rlMinMicroViaOuter" value="4mil"/>
@@
 <param name="psTop" value="-1"/>
 <param name="psBottom" value="-1"/>
-<param name="psFirst" value="-1"/>
+<param name="psFirst" value="0"/>
 <param name="psElongationLong" value="100"/>
 <param name="psElongationOffset" value="100"/>
 <param name="mvStopFrame" value="1"/>
 <param name="mvCreamFrame" value="0"/>
-<param name="mlMinStopFrame" value="4mil"/>
-<param name="mlMaxStopFrame" value="4mil"/>
+<param name="mlMinStopFrame" value="2mil"/>
+<param name="mlMaxStopFrame" value="2mil"/>
 <param name="mlMinCreamFrame" value="0mil"/>
 <param name="mlMaxCreamFrame" value="0mil"/>
-<param name="mlViaStopLimit" value="0mil"/>
+<param name="mlViaStopLimit" value="100mil"/>
 <param name="srRoundness" value="0"/>
 <param name="srMinRoundness" value="0mil"/>
@@
 <param name="checkAngle" value="0"/>
 <param name="checkFont" value="1"/>
-<param name="checkRestrict" value="1"/>
+<param name="checkRestrict" value="0"/>
 <param name="useDiameter" value="13"/>
 <param name="maxErrors" value="50"/>
@@
 <wire x1="30.48" y1="3.81" x2="31.75" y2="2.54" width="0.4064" layer="1"/>
 <wire x1="31.75" y1="2.54" x2="48.26" y2="2.54" width="0.4064" layer="1"/>
-<wire x1="29.21" y1="3.81" x2="26.67" y2="3.81" width="0.4064" layer="1"/>
-<wire x1="26.67" y1="3.81" x2="26.67" y2="23.495" width="0.4064" layer="1"/>
 <via x="26.67" y="23.495" extent="1-16" drill="0.6"/>
 <wire x1="26.67" y1="23.495" x2="25.4" y2="23.495" width="0.4064" layer="16"/>
@@
 <via x="12.065" y="40.386" extent="1-16" drill="0.6"/>
 <wire x1="12.065" y1="40.386" x2="8.0518" y2="40.386" width="0.4064" layer="1"/>
+<wire x1="29.21" y1="3.81" x2="26.67" y2="5.08" width="0.4064" layer="1"/>
+<wire x1="26.67" y1="5.08" x2="26.67" y2="23.495" width="0.4064" layer="1"/>
 </signal>
 <signal name="N$3">
@@
 <contactref element="U$1" pad="17"/>
 <contactref element="U$15" pad="1"/>
-<wire x1="29.21" y1="8.89" x2="37.465" y2="8.89" width="0.4064" layer="1"/>
-<wire x1="37.465" y1="8.89" x2="41.91" y2="13.335" width="0.4064" layer="1"/>
-<wire x1="41.91" y1="13.335" x2="46.355" y2="13.335" width="0.4064" layer="1"/>
+<wire x1="29.21" y1="8.89" x2="36.83" y2="8.89" width="0.4064" layer="1"/>
+<wire x1="36.83" y1="8.89" x2="41.275" y2="13.335" width="0.4064" layer="1"/>
+<wire x1="41.275" y1="13.335" x2="46.355" y2="13.335" width="0.4064" layer="1"/>
 <wire x1="46.355" y1="13.335" x2="48.26" y2="10.16" width="0.4064" layer="1"/>
 </signal>
@@
 <wire x1="45.72" y1="22.86" x2="44.45" y2="21.59" width="0.4064" layer="16"/>
 <wire x1="29.21" y1="31.75" x2="40.005" y2="31.75" width="0.4064" layer="1"/>
-<wire x1="40.005" y1="31.75" x2="45.085" y2="26.67" width="0.4064" layer="1"/>
-<wire x1="45.085" y1="26.67" x2="48.26" y2="26.67" width="0.4064" layer="1"/>
-<wire x1="48.26" y1="26.67" x2="48.26" y2="22.86" width="0.4064" layer="1"/>
+<wire x1="40.005" y1="31.75" x2="44.45" y2="27.305" width="0.4064" layer="1"/>
 <wire x1="44.45" y1="21.59" x2="41.91" y2="21.59" width="0.4064" layer="16"/>
+<wire x1="48.26" y1="22.86" x2="48.26" y2="24.765" width="0.4064" layer="1"/>
+<wire x1="44.45" y1="27.305" x2="45.72" y2="27.305" width="0.4064" layer="1"/>
+<wire x1="45.72" y1="27.305" x2="48.26" y2="24.765" width="0.4064" layer="1"/>
 </signal>
 <signal name="B14">
@@
 <wire x1="46.355" y1="17.78" x2="45.085" y2="19.05" width="0.4064" layer="1"/>
 <wire x1="45.085" y1="19.05" x2="45.085" y2="22.225" width="0.4064" layer="1"/>
-<wire x1="45.085" y1="22.225" x2="44.45" y2="22.86" width="0.4064" layer="1"/>
-<wire x1="44.45" y1="22.86" x2="43.18" y2="22.86" width="0.4064" layer="1"/>
-<wire x1="43.18" y1="22.86" x2="39.37" y2="26.67" width="0.4064" layer="1"/>
+<wire x1="45.085" y1="22.225" x2="43.815" y2="23.495" width="0.4064" layer="1"/>
+<wire x1="43.815" y1="23.495" x2="42.545" y2="23.495" width="0.4064" layer="1"/>
+<wire x1="42.545" y1="23.495" x2="39.37" y2="26.67" width="0.4064" layer="1"/>
 <wire x1="39.37" y1="26.67" x2="38.1" y2="26.67" width="0.4064" layer="1"/>
 </signal>
@@
 <wire x1="25.4" y1="36.83" x2="21.59" y2="36.83" width="0.4064" layer="16"/>
 <wire x1="17.78" y1="2.54" x2="19.685" y2="0.635" width="0.4064" layer="1"/>
-<wire x1="19.685" y1="0.635" x2="25.4" y2="0.635" width="0.4064" layer="1"/>
-<wire x1="25.4" y1="0.635" x2="25.4" y2="26.67" width="0.4064" layer="1"/>
-<via x="25.4" y="26.67" extent="1-16" drill="0.6" shape="square"/>
+<via x="25.4" y="26.67" extent="1-16" drill="0.6"/>
 <wire x1="25.4" y1="26.67" x2="25.4" y2="36.83" width="0.4064" layer="16"/>
+<wire x1="19.685" y1="0.635" x2="24.13" y2="0.635" width="0.4064" layer="1"/>
+<wire x1="24.13" y1="0.635" x2="25.4" y2="1.905" width="0.4064" layer="1"/>
+<wire x1="25.4" y1="1.905" x2="25.4" y2="26.67" width="0.4064" layer="1"/>
 </signal>
 <signal name="N$1">
